Commit message: new launch script (robot2 launch that works with moveit --> planning in rviz enabled)

File: src/diy_robot_wer24_moveit/srdf/robot.srdf.xacro (robot description, xacro)
@@ -1,8 +1,8 @@
 <?xml version="1.0" encoding="UTF-8"?>
 <robot xmlns:xacro="http://wiki.ros.org/xacro" name="wer24_robotarm">
-  <!-- parameters -->
-  <!-- <xacro:arg name="prefix" default="" /> -->
+  <!-- parameterspassed from the launch file -->
+  <xacro:arg name="tf_prefix" default="" />
   <xacro:include filename="$(find diy_robot_wer24_moveit)/srdf/robot_macro.srdf.xacro"/>
-  <!-- <xacro:robot_srdf name="$(arg name)" prefix="$(arg prefix)"/> -->
-  <xacro:robot_srdf/>
+  <xacro:robot_srdf tf_prefix="$(arg tf_prefix)"/>
+  <!--<xacro:robot_srdf/>-->
 </robot>

File: src/diy_robot_wer24_moveit/srdf/robot_macro.srdf.xacro (robot description, xacro)
@@ -5,5 +5,5 @@
     A URDF file must exist for this robot as well, where the joints and the links that are referenced are defined
 -->
-  <xacro:macro name="robot_srdf">
+  <xacro:macro name="robot_srdf" params="tf_prefix">
     <!--GROUPS - Representation of a set of joints and links. This can be useful for specifying DOF to plan for, defining arms, end effectors, etc-->
     <!--LINKS - When a link is specified, the parent joint of that link (if it exists) is automatically included-->
@@ -12,15 +12,17 @@
     <!--SUBGROUPS - Groups can also be formed by referencing to already defined group names-->
     <group name="wer24_robotarm">
-      <chain base_link="arm_base_link" tip_link="arm_link_6" />
+      <chain base_link="${tf_prefix}sub_subframe_link" tip_link="${tf_prefix}grip_base_link" />
     </group>
     <!--END EFFECTOR - Purpose - Represent information about an end effector.-->
     <!--VIRTUAL JOINT - Purpose - this element defines a virtual joint between a robot link and an external frame of reference (considered fixed with respect to the robot)-->
     <!--DISABLE COLLISIONS - By default it is assumed that any link of the robot could potentially come into collision with any other link in the robot. This tag disables collision checking between a specified pair of links. -->
-    <disable_collisions link1="arm_base_link" link2="arm_link_1" reason="Adjacent" />
-    <disable_collisions link1="arm_link_1" link2="arm_link_2" reason="Adjacent" />
-    <disable_collisions link1="arm_link_2" link2="arm_link_3" reason="Adjacent" />
-    <disable_collisions link1="arm_link_3" link2="arm_link_4" reason="Adjacent" />
-    <disable_collisions link1="arm_link_4" link2="arm_link_5" reason="Adjacent" />
-    <disable_collisions link1="arm_link_5" link2="arm_link_6" reason="Adjacent" />
+    <disable_collisions link1="${tf_prefix}sub_subframe_link" link2="${tf_prefix}arm_base_link" reason="Adjacent" />
+    <disable_collisions link1="${tf_prefix}arm_base_link" link2="${tf_prefix}arm_link_1" reason="Adjacent" />
+    <disable_collisions link1="${tf_prefix}arm_link_1" link2="${tf_prefix}arm_link_2" reason="Adjacent" />
+    <disable_collisions link1="${tf_prefix}arm_link_2" link2="${tf_prefix}arm_link_3" reason="Adjacent" />
+    <disable_collisions link1="${tf_prefix}arm_link_3" link2="${tf_prefix}arm_link_4" reason="Adjacent" />
+    <disable_collisions link1="${tf_prefix}arm_link_4" link2="${tf_prefix}arm_link_5" reason="Adjacent" />
+    <disable_collisions link1="${tf_prefix}arm_link_5" link2="${tf_prefix}arm_link_6" reason="Adjacent" />
+    <disable_collisions link1="${tf_prefix}arm_link_6" link2="${tf_prefix}grip_base_link" reason="Adjacent" />
   </xacro:macro>
 </robot>

Commit message: changed launch arguments

File: src/diy_robot_wer24_moveit/srdf/robot.srdf.xacro (robot description, xacro)
@@ -1,8 +1,17 @@
 <?xml version="1.0" encoding="UTF-8"?>
 <robot xmlns:xacro="http://wiki.ros.org/xacro" name="wer24_robotarm">
-  <!-- parameterspassed from the launch file -->
-  <xacro:arg name="tf_prefix" default="" />
+<!-- set some gloabal arguments (define second order namespaces to avoid name collisions)-->
+  <xacro:arg name="name" default="wer24_robotarm"/>
+  <xacro:arg name="tf_prefix" default=""/>
+  <xacro:arg name="tf_prefix_sub" default="sub_"/>
+  <xacro:arg name="tf_prefix_arm" default="arm_"/>
+  <xacro:arg name="tf_prefix_grip" default="grip_"/>
   <xacro:include filename="$(find diy_robot_wer24_moveit)/srdf/robot_macro.srdf.xacro"/>
-  <xacro:robot_srdf tf_prefix="$(arg tf_prefix)"/>
-  <!--<xacro:robot_srdf/>-->
+  <xacro:robot_srdf
+    tf_prefix="$(arg tf_prefix)"
+    tf_prefix_sub="$(arg tf_prefix_sub)"
+    tf_prefix_arm="$(arg tf_prefix_arm)"
+    tf_prefix_grip="$(arg tf_prefix_grip)"
+  >
+  </xacro:robot_srdf>
 </robot>

File: src/diy_robot_wer24_moveit/srdf/robot_macro.srdf.xacro (robot description, xacro)
@@ -5,18 +5,18 @@
     A URDF file must exist for this robot as well, where the joints and the links that are referenced are defined
 -->
-  <xacro:macro name="robot_srdf" params="tf_prefix">
+  <xacro:macro name="robot_srdf" params="tf_prefix tf_prefix_sub tf_prefix_arm tf_prefix_grip">
     <!--GROUPS - Representation of a set of joints and links. This can be useful for specifying DOF to plan for, defining arms, end effectors, etc-->
     <group name="wer24_robotarm">
-      <chain base_link="${tf_prefix}sub_subframe_link" tip_link="${tf_prefix}grip_base_link" />
+      <chain base_link="${tf_prefix}${tf_prefix_sub}subframe_link" tip_link="${tf_prefix}${tf_prefix_grip}base_link" />
     </group>
     <!--DISABLE COLLISIONS - By default it is assumed that any link of the robot could potentially come into collision with any other link in the robot. This tag disables collision checking between a specified pair of links. -->
-    <disable_collisions link1="${tf_prefix}sub_subframe_link" link2="${tf_prefix}arm_base_link" reason="Adjacent" />
-    <disable_collisions link1="${tf_prefix}arm_base_link" link2="${tf_prefix}arm_link_1" reason="Adjacent" />
-    <disable_collisions link1="${tf_prefix}arm_link_1" link2="${tf_prefix}arm_link_2" reason="Adjacent" />
-    <disable_collisions link1="${tf_prefix}arm_link_2" link2="${tf_prefix}arm_link_3" reason="Adjacent" />
-    <disable_collisions link1="${tf_prefix}arm_link_3" link2="${tf_prefix}arm_link_4" reason="Adjacent" />
-    <disable_collisions link1="${tf_prefix}arm_link_4" link2="${tf_prefix}arm_link_5" reason="Adjacent" />
-    <disable_collisions link1="${tf_prefix}arm_link_5" link2="${tf_prefix}arm_link_6" reason="Adjacent" />
-    <disable_collisions link1="${tf_prefix}arm_link_6" link2="${tf_prefix}grip_base_link" reason="Adjacent" />
+    <disable_collisions link1="${tf_prefix}${tf_prefix_sub}subframe_link" link2="${tf_prefix}arm_base_link" reason="Adjacent" />
+    <disable_collisions link1="${tf_prefix}${tf_prefix_arm}base_link" link2="${tf_prefix}${tf_prefix_arm}link_1" reason="Adjacent" />
+    <disable_collisions link1="${tf_prefix}${tf_prefix_arm}link_1" link2="${tf_prefix}${tf_prefix_arm}link_2" reason="Adjacent" />
+    <disable_collisions link1="${tf_prefix}${tf_prefix_arm}link_2" link2="${tf_prefix}${tf_prefix_arm}link_3" reason="Adjacent" />
+    <disable_collisions link1="${tf_prefix}${tf_prefix_arm}link_3" link2="${tf_prefix}${tf_prefix_arm}link_4" reason="Adjacent" />
+    <disable_collisions link1="${tf_prefix}${tf_prefix_arm}link_4" link2="${tf_prefix}${tf_prefix_arm}link_5" reason="Adjacent" />
+    <disable_collisions link1="${tf_prefix}${tf_prefix_arm}link_5" link2="${tf_prefix}${tf_prefix_arm}link_6" reason="Adjacent" />
+    <disable_collisions link1="${tf_prefix}${tf_prefix_arm}link_6" link2="${tf_prefix}${tf_prefix_grip}base_link" reason="Adjacent" />
   </xacro:macro>
 </robot>
